File: Dice/PD6/PD6v1/Main.kicad_sch (KiCad schematic)
At the start: 28 parts, among them J1 Conn_01x14, J2 Conn_01x11, U1 N52810_QFN32, U2 KXTJ3-1057, Y1 32MHz 40ppm

Commit message: Update dice boards with new battery connector.
Parts:
- R9: Manufacturer (none) -> Yageo; Manufacturer Part Number (none) -> AF0402FR-07150KL
Changed lines of the file:
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@@
       (effects (font (size 1.27 1.27)) hide)
     )
-    (property "Manufacturer" "" (id 6) (at 116.84 44.45 0)
-      (effects (font (size 1.27 1.27)) hide)
-    )
-    (property "Manufacturer Part Number" "" (id 7) (at 116.84 44.45 0)
+    (property "Manufacturer" "Yageo" (id 6) (at 116.84 44.45 0)
+      (effects (font (size 1.27 1.27)) hide)
+    )
+    (property "Manufacturer Part Number" "AF0402FR-07150KL" (id 7) (at 116.84 44.45 0)
       (effects (font (size 1.27 1.27)) hide)
     )
@@
     )
     (path "/00000000-0000-0000-0000-00005bb44a54/00000000-0000-0000-0000-00005cf24b7e"
-      (reference "U7") (unit 1) (value "74AHC1G08") (footprint "Pixels-dice:SOT-353_SC-70-5")
+      (reference "U7") (unit 1) (value "SN74LVC1G08") (footprint "Pixels-dice:SOT-353_SC-70-5")
     )
     (path "/00000000-0000-0000-0000-00005bb44a54/00000000-0000-0000-0000-00006143ac96"
