File: Dice/PD6/PD6v2/LEDs.kicad_sch (KiCad schematic)
At the start: 25 parts

Commit message: Updating D8 and D10 boards, new antenna, etc...
Parts:
- W22: Generic OK (none) -> N/A
Changed lines of the file:
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@@
     )
     (property "Datasheet" "" (id 3) (at 30.48 45.72 0))
+    (property "Generic OK" "N/A" (id 4) (at 25.4 45.72 0)
+      (effects (font (size 1.27 1.27)) hide)
+    )
     (pin "1")
   )
