File: Dice/D6/D6v4/Power.kicad_sch (KiCad schematic)
At the start: 11 parts, among them U4 ME6215, U6 MT9700, U7 SN74LVC1G08, U8 TMR1366

Commit message: Updated all remaining boards to match D20V15 (D6, PD6, D8, D10 and D12)
Parts:
- C16, C9: Manufacturer Part Number GRM155R61A106ME11D -> GRM155R61A106ME44D
Changed lines of the file:
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@@
       (effects (font (size 1.27 1.27)) hide)
     )
-    (property "Manufacturer Part Number" "GRM155R61A106ME11D" (id 7) (at 130.81 132.08 0)
+    (property "Manufacturer Part Number" "GRM155R61A106ME44D " (id 7) (at 130.81 132.08 0)
       (effects (font (size 1.27 1.27)) hide)
     )
@@
       (effects (font (size 1.27 1.27)) hide)
     )
-    (property "Manufacturer Part Number" "GRM155R61A106ME11D" (id 7) (at 191.77 67.31 0)
+    (property "Manufacturer Part Number" "GRM155R61A106ME44D " (id 7) (at 191.77 67.31 0)
       (effects (font (size 1.27 1.27)) hide)
     )
