File: Dice/D6/D6v5/wireless.kicad_sch (KiCad schematic)
At the start: 29 parts, among them J3 Conn_01x02, P5 COILA, P6 COILB, U3 PJ75AL50SA, U5 MCP73832T-2ACI/OT

Commit message: Update Dice FPC and LCC PCB
Parts:
- P5, P6: footprint TestPoint:TestPoint_THTPad_D1.5mm_Drill0.7mm -> Pixels-dice:TestPoint_THTPad_D1.5mm_Drill0.7mm_nosilk
Changed lines of the file:
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@@
       (effects (font (size 1.27 1.27)))
     )
-    (property "Footprint" "TestPoint:TestPoint_THTPad_D1.5mm_Drill0.7mm" (at 57.15 68.58 0)
+    (property "Footprint" "Pixels-dice:TestPoint_THTPad_D1.5mm_Drill0.7mm_nosilk" (at 57.15 68.58 0)
       (effects (font (size 1.27 1.27)) hide)
     )
@@
       (effects (font (size 1.27 1.27)))
     )
-    (property "Footprint" "TestPoint:TestPoint_THTPad_D1.5mm_Drill0.7mm" (at 57.15 66.04 0)
+    (property "Footprint" "Pixels-dice:TestPoint_THTPad_D1.5mm_Drill0.7mm_nosilk" (at 57.15 66.04 0)
       (effects (font (size 1.27 1.27)) hide)
     )
