File: Large Charging Case/LCCV3.6/multiplexed_chargers.kicad_sch (KiCad schematic)
At the start: 26 parts, among them U17 74HC4051PW, U18 LM2902, U19 74HCT259PW, U20 LM2902

Commit message: More board updates
Parts:
- U18: LCSC Part Number C46864 -> (none); Manufacturer Texas Instrument -> XINLUDA; Manufacturer Part Number LM2902PWR -> XL2902-TS
- U20: value LM2902 -> XL2902-TS; LCSC Part Number C46864 -> (none); Manufacturer Texas Instrument -> XINLUDA; Manufacturer Part Number LM2902PWR -> XL2902-TS
Changed lines of the file:
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@@
       (effects (font (size 1.27 1.27)) (justify left))
     )
-    (property "Value" "LM2902" (at 75.565 36.1566 0)
+    (property "Value" "XL2902-TS" (at 75.565 36.1566 0)
       (effects (font (size 1.27 1.27)) (justify left))
     )
@@
       (effects (font (size 1.27 1.27)) hide)
     )
-    (property "Datasheet" "http://www.ti.com/lit/ds/symlink/lm2902-n.pdf" (at 78.74 29.21 0)
-      (effects (font (size 1.27 1.27)) hide)
-    )
-    (property "LCSC Part Number" "C46864" (at 77.47 34.29 0)
-      (effects (font (size 1.27 1.27)) hide)
-    )
-    (property "Manufacturer" "Texas Instrument" (at 77.47 34.29 0)
-      (effects (font (size 1.27 1.27)) hide)
-    )
-    (property "Manufacturer Part Number" "LM2902PWR" (at 77.47 34.29 0)
+    (property "Datasheet" "" (at 78.74 29.21 0)
+      (effects (font (size 1.27 1.27)) hide)
+    )
+    (property "LCSC Part Number" "" (at 77.47 34.29 0)
+      (effects (font (size 1.27 1.27)) hide)
+    )
+    (property "Manufacturer" "XINLUDA" (at 77.47 34.29 0)
+      (effects (font (size 1.27 1.27)) hide)
+    )
+    (property "Manufacturer Part Number" "XL2902-TS" (at 77.47 34.29 0)
       (effects (font (size 1.27 1.27)) hide)
     )
@@
       (effects (font (size 1.27 1.27)) hide)
     )
-    (property "Datasheet" "http://www.ti.com/lit/ds/symlink/lm2902-n.pdf" (at 66.04 29.21 0)
-      (effects (font (size 1.27 1.27)) hide)
-    )
-    (property "LCSC Part Number" "C46864" (at 64.77 34.29 0)
-      (effects (font (size 1.27 1.27)) hide)
-    )
-    (property "Manufacturer" "Texas Instrument" (at 64.77 34.29 0)
-      (effects (font (size 1.27 1.27)) hide)
-    )
-    (property "Manufacturer Part Number" "LM2902PWR" (at 64.77 34.29 0)
-      (effects (font (size 1.27 1.27)) hide)
-    )
+    (property "Datasheet" "" (at 66.04 29.21 0)
+      (effects (font (size 1.27 1.27)) hide)
+    )
+    (property "LCSC Part Number" "" (at 64.77 34.29 0)
+      (effects (font (size 1.27 1.27)) hide)
+    )
+    (property "Manufacturer" "XINLUDA" (at 64.77 34.29 0)
+      (effects (font (size 1.27 1.27)) hide)
+    )
+    (property "Manufacturer Part Number" "XL2902-TS" (at 64.77 34.29 0)
+      (effects (font (size 1.27 1.27)) hide)
+    )
