File: Dice/D10/D10v5/Main.kicad_sch (KiCad schematic)
At the start: 33 parts, among them J1 Conn_01x14, J2 Conn_01x04, J4 DNP, U1 N52810_QFN32, U2 KXTJ3-1057, Y1 32MHz 40ppm

Commit message: Update BOM on all dice. Make sure testpins are excluded from BOM in all dice. Slight Tweak to D8 layout.
Parts:
- J1, J2, W1, W10, W2, W5, W6, W7, W8, W9: now left out of the parts list
Changed lines of the file:
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@@
   )
   (symbol (lib_id "Pixels-dice:TEST_1P-conn") (at 160.02 116.84 0) (unit 1)
-    (in_bom yes) (on_board yes) (dnp no)
+    (in_bom no) (on_board yes) (dnp no)
     (property "Reference" "W1" (at 157.48 109.22 0)
       (effects (font (size 1.27 1.27)) (justify left))
@@
   )
   (symbol (lib_id "Pixels-dice:TEST_1P-conn") (at 162.56 116.84 0) (unit 1)
-    (in_bom yes) (on_board yes) (dnp no)
+    (in_bom no) (on_board yes) (dnp no)
     (property "Reference" "W2" (at 162.56 109.22 0)
       (effects (font (size 1.27 1.27)) (justify left))
@@
   )
   (symbol (lib_id "Pixels-dice:TEST_1P-conn") (at 88.9 152.4 270) (unit 1)
-    (in_bom yes) (on_board yes) (dnp no)
+    (in_bom no) (on_board yes) (dnp no)
     (property "Reference" "W5" (at 93.98 151.13 90)
       (effects (font (size 1.27 1.27)) (justify left))
@@
   )
   (symbol (lib_id "Pixels-dice:TEST_1P-conn") (at 149.86 147.32 0) (unit 1)
-    (in_bom yes) (on_board yes) (dnp no)
+    (in_bom no) (on_board yes) (dnp no)
     (property "Reference" "W7" (at 146.05 143.51 0)
       (effects (font (size 1.27 1.27)) (justify left))
@@
   )
   (symbol (lib_id "Pixels-dice:TEST_1P-conn") (at 157.48 147.32 0) (unit 1)
-    (in_bom yes) (on_board yes) (dnp no)
+    (in_bom no) (on_board yes) (dnp no)
     (property "Reference" "W8" (at 153.67 143.51 0)
       (effects (font (size 1.27 1.27)) (justify left))
@@
   )
   (symbol (lib_id "Pixels-dice:TEST_1P-conn") (at 165.1 147.32 0) (unit 1)
-    (in_bom yes) (on_board yes) (dnp no)
+    (in_bom no) (on_board yes) (dnp no)
     (property "Reference" "W9" (at 161.29 143.51 0)
       (effects (font (size 1.27 1.27)) (justify left))
@@
   )
   (symbol (lib_id "Connector_Generic:Conn_01x14") (at 229.87 44.45 0) (unit 1)
-    (in_bom yes) (on_board yes) (dnp no)
+    (in_bom no) (on_board yes) (dnp no)
     (property "Reference" "J1" (at 231.902 44.6532 0)
       (effects (font (size 1.27 1.27)) (justify left))
@@
   )
   (symbol (lib_id "Connector_Generic:Conn_01x04") (at 269.24 44.45 0) (unit 1)
-    (in_bom yes) (on_board yes) (dnp no) (fields_autoplaced)
+    (in_bom no) (on_board yes) (dnp no) (fields_autoplaced)
     (property "Reference" "J2" (at 271.78 44.4499 0)
       (effects (font (size 1.27 1.27)) (justify left))
@@
   )
   (symbol (lib_id "Pixels-dice:TEST_1P-conn") (at 139.7 100.33 90) (unit 1)
-    (in_bom yes) (on_board yes) (dnp no)
+    (in_bom no) (on_board yes) (dnp no)
     (property "Reference" "W6" (at 132.08 102.87 0)
       (effects (font (size 1.27 1.27)) (justify left))
@@
   )
   (symbol (lib_id "Pixels-dice:TEST_1P-conn") (at 142.24 100.33 270) (unit 1)
-    (in_bom yes) (on_board yes) (dnp no)
+    (in_bom no) (on_board yes) (dnp no)
     (property "Reference" "W10" (at 149.86 100.33 0)
       (effects (font (size 1.27 1.27)) (justify left))
