File: Dice/D12/D12v5/wireless.kicad_sch (KiCad schematic)
At the start: 29 parts, among them J3 Conn_01x02, P5 COILA, P6 COILB, U3 PJ75BL50SA, U5 MCP73832T-2ACI/OT

Commit message: Update BOM on all dice. Make sure testpins are excluded from BOM in all dice. Slight Tweak to D8 layout.
Parts:
- J3, P5, P6, W13, W14, W15, W16, W17, W19, W20, W3, W4: now left out of the parts list
Changed lines of the file:
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@@
   )
   (symbol (lib_id "Pixels-dice:TEST_1P-conn") (at 120.65 49.53 0) (unit 1)
-    (in_bom yes) (on_board yes) (dnp no)
+    (in_bom no) (on_board yes) (dnp no)
     (property "Reference" "W16" (at 122.1232 46.482 0)
       (effects (font (size 1.27 1.27)) (justify left))
@@
   )
   (symbol (lib_id "Pixels-dice:TEST_1P-conn") (at 54.61 129.54 90) (unit 1)
-    (in_bom yes) (on_board yes) (dnp no)
+    (in_bom no) (on_board yes) (dnp no)
     (property "Reference" "W13" (at 51.562 128.0668 0)
       (effects (font (size 1.27 1.27)) (justify left))
@@
   )
   (symbol (lib_id "Pixels-dice:TEST_1P-conn") (at 182.88 62.23 90) (unit 1)
-    (in_bom yes) (on_board yes) (dnp no)
+    (in_bom no) (on_board yes) (dnp no)
     (property "Reference" "W3" (at 180.34 67.31 90)
       (effects (font (size 1.27 1.27)) (justify left))
@@
   )
   (symbol (lib_id "Pixels-dice:TEST_1P-conn") (at 172.72 129.54 90) (unit 1)
-    (in_bom yes) (on_board yes) (dnp no)
+    (in_bom no) (on_board yes) (dnp no)
     (property "Reference" "W4" (at 169.672 128.0668 0)
       (effects (font (size 1.27 1.27)) (justify left))
@@
   )
   (symbol (lib_id "Pixels-dice:TEST_1P-conn") (at 222.25 69.85 0) (unit 1)
-    (in_bom yes) (on_board yes) (dnp no)
+    (in_bom no) (on_board yes) (dnp no)
     (property "Reference" "W17" (at 220.98 64.77 90)
       (effects (font (size 1.27 1.27)) (justify left))
@@
   )
   (symbol (lib_id "Connector_Generic:Conn_01x02") (at 256.54 57.15 0) (unit 1)
-    (in_bom yes) (on_board yes) (dnp no)
+    (in_bom no) (on_board yes) (dnp no)
     (property "Reference" "J3" (at 258.572 57.3532 0)
       (effects (font (size 1.27 1.27)) (justify left))
@@
   )
   (symbol (lib_id "Pixels-dice:TEST_1P-conn") (at 120.65 68.58 180) (unit 1)
-    (in_bom yes) (on_board yes) (dnp no)
+    (in_bom no) (on_board yes) (dnp no)
     (property "Reference" "W19" (at 122.1232 69.2658 0)
       (effects (font (size 1.27 1.27)) (justify right))
@@
   )
   (symbol (lib_id "Pixels-dice:TEST_1P-conn") (at 237.49 46.99 0) (unit 1)
-    (in_bom yes) (on_board yes) (dnp no)
+    (in_bom no) (on_board yes) (dnp no)
     (property "Reference" "W14" (at 236.22 41.91 90)
       (effects (font (size 1.27 1.27)) (justify left))
@@
   )
   (symbol (lib_id "Connector_Generic:Conn_01x01") (at 57.15 68.58 180) (unit 1)
-    (in_bom yes) (on_board yes) (dnp no)
+    (in_bom no) (on_board yes) (dnp no)
     (property "Reference" "P6" (at 53.34 68.58 0)
       (effects (font (size 1.27 1.27)))
@@
   )
   (symbol (lib_id "Connector_Generic:Conn_01x01") (at 57.15 66.04 180) (unit 1)
-    (in_bom yes) (on_board yes) (dnp no)
+    (in_bom no) (on_board yes) (dnp no)
     (property "Reference" "P5" (at 53.34 66.04 0)
       (effects (font (size 1.27 1.27)))
@@
   )
   (symbol (lib_id "Pixels-dice:TEST_1P-conn") (at 114.3 129.54 90) (unit 1)
-    (in_bom yes) (on_board yes) (dnp no)
+    (in_bom no) (on_board yes) (dnp no)
     (property "Reference" "W20" (at 111.252 128.0668 0)
       (effects (font (size 1.27 1.27)) (justify left))
@@
   )
   (symbol (lib_id "Pixels-dice:TEST_1P-conn") (at 161.29 49.53 0) (unit 1)
-    (in_bom yes) (on_board yes) (dnp no)
+    (in_bom no) (on_board yes) (dnp no)
     (property "Reference" "W15" (at 162.7632 46.482 0)
       (effects (font (size 1.27 1.27)) (justify left))
