File: Dice/Super6/Super6V1/UVLEDs.kicad_sch (KiCad schematic)
At the start: 24 parts, among them U9 MT9700

Commit message: D10V5, D20V16 and Super6V1
Parts:
- removed D11, D16, D49, D50, D51: UV LED, Pixels-dice:MHP1016UVACT, symbol Device:LED
- removed R14, R17, R22, R23, R24: 33R 1%, Resistor_SMD:R_0402_1005Metric, symbol Device:R
