File: Dice/D6/D6v9/Power.kicad_sch (KiCad schematic)
At the start: 12 parts, among them U4 ME6215, U6 MT9700, U7 SN74LVC1G08, U8 VCS2373S, U8-alt1 VCS2373S

Commit message: D6V9 and new Jigs
Parts:
- removed U8-alt1: VCS2373S, Pixels-dice:SOT-23, symbol Pixels-dice:TMR1366
- added U9: VCS2373S, Package_TO_SOT_SMD:SOT-23, symbol Pixels-dice:TMR1366
- U8: footprint Pixels-dice:SOT-23 -> Package_TO_SOT_SMD:SOT-23
Connections:
- net +BATT: now also U9.1 (VCC)
- net GND: now also U9.3 (GND)
- net MAG1_: now also U9.2 (OUT)
Other:
- title: Pixels D20 Schematic, Power -> Pixels D6 Schematic, Main
