File: JIGs/LCC Jig Plug/main.kicad_pcb (KiCad board)
At the start: 2 copper layers, 19.8 x 11 mm, 18 parts, among them J1 Conn_01x04, J2 Conn_01x03, P1 COILA, P2 COILB, U1 PJ75BL50SA, U2 MCP73832T-2ACI/OT

Commit message: LCCV3.8 and Jig updates
Parts:
- U1: value PJ75BL50SA -> PJ75AL50SA

Commit message: D6V9 and new Jigs
Connections:
- J1 pad 3: GND -> +5V
Routing:
- net GND: track 45.1 -> 38.8 mm, vias 4 -> 5
- net +5V: track 9.04 -> 14.5 mm, vias 0 -> 1
