File: Dice/Puck/PuckV2 Test/Main.kicad_sch (KiCad schematic)
At the start: 31 parts, among them J2 Conn_01x04, J3 Conn_01x09, J4 DNP, J5 Conn_02x03_Odd_Even, U1 NRF52810-CAAA-R, U11 SC7A20HTR, U4 M24C02-FMH6TG, U8 SL1605, Y1 32MHz 40ppm

Commit message: more board file updates
Parts:
- removed U11: SC7A20HTR, Package_LGA:LGA-12_2x2mm_P0.5mm, symbol Pixels-dice:SC7A20HTR
- removed U8: SL1605, Package_TO_SOT_SMD:SOT-553, symbol Pixels-dice:SL1605
- added U11: KXTJ3-1057, Package_LGA:LGA-12_2x2mm_P0.5mm, symbol Pixels-dice:KXTJ3-1057
- W7, W8, W9: footprint Connector_PinHeader_2.54mm:PinHeader_1x01_P2.54mm_Vertical -> Pixels-dice:TEST_PIN
Connections:
- net ACC_INT: now also U11.5 (INT)
- net GND: now also U11.6 (GND), U11.8 (GND), U11.9 (GND)
- net MAG2_: no longer J3.7 (Pin_7), U1.F2 (P0.21)
- net SCL: now also U11.12 (SCL)
- net SDA: now also U11.2 (SDA)
- net VDD: now also U11.1 (ADDR), U11.10 (VDD), U11.11 (IO_VDD), U11.3 (IO_VDD), U11.7 (VDD)
- net MAG1_ renamed OPT_IO
- net OPT_IO: now also J3.7 (Pin_7)
- no-connect marks 4 -> 5
