File: Dice/Pyre/PyreV1/wireless.kicad_sch (KiCad schematic)
At the start: 36 parts, among them J1 Conn_01x02, P5 COILA, P6 COILB, Q1 ZSPT-Z1608C-06F-Z4, U10 WAS3157D-6/TR, U3 TPS715, U7 DS6101, U9 XT4051

Commit message: more board file updates
Parts:
- removed J1: Conn_01x02, Pixels-dice:Batt_409090_Tabs, symbol Connector_Generic:Conn_01x02
- removed Q1: ZSPT-Z1608C-06F-Z4, Diode_SMD:D_0603_1608Metric, symbol Device:Q_Photo_NPN
- removed R5: 10k 1%, Resistor_SMD:R_0201_0603Metric, symbol Device:R
- removed U9: XT4051, Package_TO_SOT_SMD:SOT-553, symbol Pixels-dice:XT4051
- removed W18: PROG, Pixels-dice:TEST_PIN, symbol Pixels-dice:TEST_1P-conn
- removed W26: PHOTO, Pixels-dice:TEST_PIN, symbol Pixels-dice:TEST_1P-conn
- added J3: Conn_01x02, Pixels-dice:Batt 1025 Tabs, symbol Connector_Generic:Conn_01x02
- added U11: WS4518D, Pixels-dice:DFN-6-1EP_2x2mm_P0.65mm_EP1x1.6mm, symbol Pixels-dice:WS4518D
- added W2: PROG, Pixels-dice:TEST_PIN, symbol Pixels-dice:TEST_1P-conn
- added W5: SM, Pixels-dice:TEST_PIN, symbol Pixels-dice:TEST_1P-conn
- C13: LCSC Part # (none) -> C6119795; LCSC Part Number C6119795 -> (none)
- C15: LCSC Part # (none) -> C6119863; LCSC Part Number C6119863 -> (none)
- C19: LCSC Part # (none) -> C97906; LCSC Part Number C97906 -> (none)
- C21, C22: Alternate LCSC Part # (none) -> C76941; JLCPCB Part Number C76941 -> (none); LCSC Part # (none) -> C7503521; LCSC Part Number C7503521 -> (none)
- C23: LCSC Part # (none) -> C6119757; LCSC Part Number C6119757 -> (none)
- D1: LCSC Part # (none) -> C96225; LCSC Part Number C96225 -> (none)
- P5, P6: footprint Pixels-dice:COIL_CON -> Pixels-dice:TestPoint_THTPad_D1.5mm_Drill0.7mm_nosilk
- R1, R2, R7: Alternate LCSC Part # (none) -> C166210; JLCPCB Part Number C166210 -> (none); LCSC Part # (none) -> C423545; LCSC Part Number C423545 -> (none)
- R12: LCSC Part # (none) -> C965307; LCSC Part Number C965307 -> (none)
- R4: LCSC Part # (none) -> C473048; LCSC Part Number C473048 -> (none)
- R6: value 5.6k 1% -> 33k 1%; LCSC Part # (none) -> C473534; LCSC Part Number C965305 -> (none); Part Number NQ01WMJ0562TEE -> 0201WMF3302TEE
- R8: LCSC Part # (none) -> C423797; LCSC Part Number C423797 -> (none)
- R9: LCSC Part # (none) -> C270364; LCSC Part Number C270364 -> (none)
- TH1: LCSC Part # (none) -> C107344; LCSC Part Number C107344 -> (none)
- U10: LCSC Part # (none) -> C2939860; LCSC Part Number C2939860 -> (none)
- U3: Alternate LCSC Part # (none) -> C571193; JLCPCB Part Number C571193 -> (none); LCSC Part # (none) -> C7202975; LCSC Part Number C7202975 -> (none)
- U7: LCSC Part # (none) -> C7499469; LCSC Part Number C7499469 -> (none)
Connections:
- net +5V: now also U11.3 (VCC)
- net +BATT: now also J3.1 (Pin_1), U11.4 (BAT)
- net B-: now also J3.2 (Pin_2)
- net GND: now also R6.2, U11.2 (GND), U11.6 (TEMP), U11.7 (PAD)
- net PROG: now also R6.1, U11.1 (PROG), W2.1; no longer R6.2
- net SM: now also W5.1
- net STAT: now also U11.5 (CHRG)
- net TH1: now reaches R9.2, TH1.1, U10.1 (B0), W20.1
- net OPT_A2D: now reaches U10.3 (B1)
Other:
- note removed: "~35mA Max Charge Rate"
- moved on the sheet: P5, P6
