File: Hex Charger/Hex Charger V1.1/main.kicad_sch (KiCad schematic)
At the start: 20 parts, among them J1 USB_C_Receptacle_USB2.0, U1 MT3608B, U9 SSP61CN4802MR

Commit message: Updated boards
Parts:
- R26, R27: value 100 -> 200R 5%; LCSC Part # C25076 -> C25087; Part Number 0402WGF1000TCE -> 0402WGF2000TCE
Changed lines of the file:
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@@
 			)
 		)
-		(property "Value" "100"
+		(property "Value" "200R 5%"
 			(at 147.066 120.65 0)
 			(effects
@@
 			)
 		)
-		(property "Part Number" "0402WGF1000TCE"
+		(property "Part Number" "0402WGF2000TCE"
 			(at 148.59 119.38 0)
 			(effects
@@
 			)
 		)
-		(property "LCSC Part #" "C25076"
+		(property "LCSC Part #" "C25087"
 			(at 148.59 119.38 0)
 			(effects
@@
 			)
 		)
-		(property "Value" "100"
+		(property "Value" "200R 5%"
 			(at 159.004 120.65 0)
 			(effects
@@
 			)
 		)
-		(property "Part Number" "0402WGF1000TCE"
+		(property "Part Number" "0402WGF2000TCE"
 			(at 153.67 119.38 0)
 			(effects
@@
 			)
 		)
-		(property "LCSC Part #" "C25076"
-			(at 153.67 119.38 0)
-			(effects
+		(property "LCSC Part #" "C25087"
+			(at 153.67 119.38 0)
+			(effects
