File: Dice/D20/D20v17/Power.kicad_sch (KiCad schematic)
At the start: 9 parts, among them U5 AW35122, U6 ME6230

Commit message: Updated schematic Titles in D20V17 and likes, added 12mm D6 and Charging Jig
Other:
- title: Pixels D20 Schematic, Main -> Pixels D20V17 Schematic, Main
Changed lines of the file:
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@@
 	(paper "A4")
 	(title_block
-		(title "Pixels D20 Schematic, Main")
-		(date "2022-08-26")
+		(title "Pixels D20V17 Schematic, Main")
+		(date "2025-10-10")
 		(rev "13")
 		(company "Systemic Games, LLC")
