File: Dice/D8/D8v8/wireless.kicad_sch (KiCad schematic)
At the start: 34 parts, among them J3 Conn_01x02, P5 COILA, P6 COILB, U10 WAS3157D-6/TR, U3 PJ75BL50SA, U7 DS6101, U9 XT4051

Commit message: Updated schematic Titles in D20V17 and likes, added 12mm D6 and Charging Jig
Other:
- title: Pixels D20 Schematic, Main -> Pixels D8V8 Schematic, Main
Changed lines of the file:
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@@
 	(paper "A4")
 	(title_block
-		(title "Pixels D20 Schematic, Main")
-		(date "2022-08-26")
+		(title "Pixels D8V8 Schematic, Main")
+		(date "2025-10-10")
 		(rev "13")
 		(company "Systemic Games, LLC")
