File: Dice/D00/D00V3/LEDs.kicad_sch (KiCad schematic)
At the start: 22 parts

Commit message: Updated latest FPC versions
Other:
- title: Pixels D20 Schematic, LEDs -> Pixels D00 Schematic, Main
Changed lines of the file:
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@@
 	(paper "A4")
 	(title_block
-		(title "Pixels D20 Schematic, LEDs")
-		(date "2020-04-13")
-		(rev "2")
+		(title "Pixels D00 Schematic, Main")
+		(date "2025-10-12")
+		(rev "3")
 		(company "Systemic Games, LLC")
 	)
