File: Dice/D6/D6v11/wireless.kicad_sch (KiCad schematic)
At the start: 31 parts, among them J3 Conn_01x02, P5 COILA, P6 COILB, U3 PJ75BL50SA, U7 DS6101, U9 XT4051

Commit message: Updated latest FPC versions
Other:
- title: Pixels D20 Schematic, Main -> Pixels D6 Schematic, Main
Changed lines of the file:
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@@
 	(paper "A4")
 	(title_block
-		(title "Pixels D20 Schematic, Main")
-		(date "2022-08-26")
-		(rev "13")
+		(title "Pixels D6 Schematic, Main")
+		(date "2025-10-12")
+		(rev "11")
 		(company "Systemic Games, LLC")
 		(comment 1 "Wireless Charging Circuitry")
