File: Dice/D6_12mm/D6_12mm_V1/wireless.kicad_sch (KiCad schematic)
At the start: 44 parts, among them J3 Conn_01x02, P5 COILA, P6 COILB, U3 MG78L05AT3, U5 MT9700, U6 ME6212C30M5G, U7 DS6101, U8 MGH303A1T3, U9 TP4054(LX)

Commit message: more tweaks to d6_12mm and charging jig
Parts:
- U3: Part Number (none) -> MG78L05AT3
Changed lines of the file:
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@@
+			)
+		)
+		(property "Part Number" "MG78L05AT3"
+			(at 137.16 34.29 0)
+			(effects
+				(font
+					(size 1.27 1.27)
+				)
+				(hide yes)
 			)
 		)
